Commit message: Mesh files updated

File: src/onebot_description/urdf/onebot.urdf.xacro (robot description, xacro)
@@ -29,4 +29,11 @@
         </collision>
     </link>
+    <link   name =  "base_footprint"/>
+    <joint name = "base_joint"  type = "fixed">
+        <parent link="base_footprint"/>
+        <child link="base_link"/>
+        <origin xyz="0.0 0.0 0.09188" rpy="0 0 0" />
+        <axis xyz="0 1 0" rpy="0 0 0" />
+    </joint>
     <xacro:caster caster_prefix="rear" parent_link="base_link" >
         <origin xyz="-0.20 0.0 -0.02533" rpy="0 0 0" />

Commit message: Changed package name

File: src/onebot_description/urdf/onebot.urdf.xacro (robot description, xacro)
@@ -2,27 +2,36 @@
 <robot  xmlns:xacro="http://ros.org/wiki/xacro"
         name="onebot" >
-    <xacro:include filename="$(find onebot_description)/urdf/caster/caster.urdf.xacro" />
-    <xacro:include filename="$(find onebot_description)/urdf/wheel/wheel.urdf.xacro" />
+    <xacro:include filename="$(find onebot_description)/urdf/caster.urdf.xacro" />
+    <xacro:include filename="$(find onebot_description)/urdf/wheel.urdf.xacro" />
     <xacro:include filename="$(find onebot_description)/urdf/materials.urdf.xacro" />
-    <xacro:arg name="mesh_enabled" default="true" />
+    <xacro:arg name="mesh_enabled" default="false" />
+    <xacro:arg name="robot_namespace" default="/"/>
     <link   name = "base_link">
         <inertial>
-            <origin xyz="-0.10 0 -0.02279" rpy="0 0 0"/>
-            <mass value="1.49159"/>
-            <inertia ixx="0.00888242278" ixy="0.0" ixz="0.00087302844"
-                    iyy="0.00695847544" iyz="-0.0"
-                    izz="0.013496920"/>
+            <origin xyz="-0.108 0 -0.02579" rpy="0 0 0"/>
+            <mass value="3.978"/>
+            <inertia ixx="0.021858680" ixy="0.0" ixz="0.010020353"
+                    iyy="0.078572349" iyz="-0.0"
+                    izz="0.091971324"/>
         </inertial>
         <visual>
-            <origin xyz="0 0 0" rpy="0 0 0" />
-            <geometry>
-                <mesh filename="package://onebot_description/meshes/base_link.dae" />
-            </geometry>
-            <material name="Blue" />
+            <xacro:if value="$(arg mesh_enabled)">
+                <origin xyz="0 0 0" rpy="0 0 0" />
+                <geometry>
+                    <mesh filename="package://onebot_description/meshes/base_link.dae" />
+                </geometry>
+            </xacro:if>
+            <xacro:unless value="$(arg mesh_enabled)">
+                <origin xyz="-0.125 0 -0.01" rpy="0 0 0" />
+                <geometry>
+                    <box size="0.25 0.25 0.02" />
+                </geometry>
+                <material name="Blue" />
+            </xacro:unless>
         </visual>
         <collision>
-            <origin xyz="0 0 0" rpy="0 0 0" />
+            <origin xyz="-0.125 0 -0.01" rpy="0 0 0" />
             <geometry>
-                <mesh filename="package://onebot_description/meshes/base_link.dae" />
+                <box size="0.25 0.25 0.02" />
             </geometry>
             <material name="Blue" />
@@ -47,5 +56,5 @@
     <gazebo>
         <plugin name="gazebo_ros_control" filename="libgazebo_ros_control.so">
-        <robotNamespace>/</robotNamespace>
+        <robotNamespace>$(arg robot_namespace)</robotNamespace>
         <legacyModeNS>true</legacyModeNS>
         </plugin>

File: src/onebot_description/urdf/wheel.urdf.xacro (robot description, xacro)
@@ -1,8 +1,4 @@
 <?xml version="1.0"?>
 <robot name="wheel" xmlns:xacro="http://ros.org/wiki/xacro" >
-	<!-- Wheel Dimensions -->
-    <xacro:property name="wheel_length" value="0.032" />
-    <xacro:property name="wheel_radius" value="0.062" />
-    <xacro:property name="wheel_separation" value="0.503" />
 	<xacro:property name="wheel_kp" value="600000" />
     <xacro:property name="wheel_kd" value="3" />
@@ -19,5 +15,5 @@
 			</inertial>
 			<visual>
-				<material name="Blue"/>
+				<material name="Green"/>
 				<xacro:if value="$(arg mesh_enabled)">
 					<origin xyz="0 0 0" rpy="0 0 ${M_PI/2}" />
@@ -34,5 +30,5 @@
 			</visual>
 			<collision>
-				<material name="Blue"/>
+				<material name="Green"/>
 				<origin xyz="0 0 0" rpy="${M_PI/2} 0 0" />
 				<geometry>
